Commit message: Fix stl and attach arm to robot

File: turtlebot3_description/urdf/turtlebot3_burger.urdf.xacro (robot description, xacro)
@@ -113,10 +113,11 @@
   </joint>
   <link name="imu_link"/>
-  <joint name="scan_joint" type="fixed">
+ <joint name="scan_joint" type="fixed">
     <parent link="base_link"/>
-    <child link="base_scan"/>
+    <child link="arm_link"/>
     <origin xyz="-0.032 0 0.172" rpy="0 0 0"/>
   </joint>
-  <link name="base_scan">
+<link name="arm_link" />
+ <!-- <link name="base_scan">
     <visual>
       <origin xyz="0 0 0.0" rpy="0 0 0"/>
@@ -139,4 +140,8 @@
                izz="0.001" />
     </inertial>
-  </link>
+  </link> -->
+   <include filename="$(find turtlebot_arm_description)/urdf/$(optenv TURTLEBOT_ARM1 pincher)_arm.urdf.xacro" />
+   <turtlebot_arm parent="arm_link" color="Gray" gripper_color="Gray" pincher_gripper="true" turtlebot_gripper="false">
+      <origin xyz="0 0 0"/>
+   </turtlebot_arm>
 </robot>

Commit message: Arm added on top of lidar

File: turtlebot3_description/urdf/turtlebot3_burger.urdf.xacro (robot description, xacro)
@@ -3,4 +3,7 @@
   <xacro:include filename="$(find turtlebot3_description)/urdf/common_properties.xacro"/>
   <xacro:include filename="$(find turtlebot3_description)/urdf/turtlebot3_burger.gazebo.xacro"/>
+  <xacro:property name="AX12_HEIGHT" value="0.0385"/>
+  <xacro:property name="AX12_WIDTH" value="0.038"/>
+  <xacro:property name="AX12_LENGTH" value="0.050"/>
   <link name="base_footprint"/>
   <joint name="base_joint" type="fixed">
@@ -115,9 +118,8 @@
  <joint name="scan_joint" type="fixed">
     <parent link="base_link"/>
-    <child link="arm_link"/>
+    <child link="base_scan"/>
     <origin xyz="-0.032 0 0.172" rpy="0 0 0"/>
   </joint>
-<link name="arm_link" />
- <!-- <link name="base_scan">
+  <link name="base_scan">
     <visual>
       <origin xyz="0 0 0.0" rpy="0 0 0"/>
@@ -140,8 +142,35 @@
                izz="0.001" />
     </inertial>
-  </link> -->
+  </link>
+  <joint name="arm_joint" type="fixed">
+    <parent link="base_link" />
+    <child link="base_arm" />
+    <origin xyz="-0.036 0.04 0.2385" rpy="0 0 0"/>
+  </joint>
+  <link name="base_arm">
+    <visual>
+      <origin xyz="0 0 0.0" rpy="0 0 0"/>
+      <geometry>
+        <mesh filename="package://turtlebot3_description/meshes/bases/burger_arm_base.stl" scale="0.01 0.01 0.01"/>
+      </geometry>
+      <material name="dark"/>
+    </visual>
+    <collision>
+      <origin xyz="0 -0.039 -0.049" rpy="0 0 0"/>
+      <geometry>
+        <box size="0.137 0.137 0.098" />
+      </geometry>
+    </collision>
+    <inertial>
+      <mass value="0.114" />
+      <origin xyz="0 0 0" />
+      <inertia ixx="0.001" ixy="0.0" ixz="0.0"
+               iyy="0.001" iyz="0.0"
+               izz="0.001" />
+    </inertial>
+  </link>
    <include filename="$(find turtlebot_arm_description)/urdf/$(optenv TURTLEBOT_ARM1 pincher)_arm.urdf.xacro" />
-   <turtlebot_arm parent="arm_link" color="Gray" gripper_color="Gray" pincher_gripper="true" turtlebot_gripper="false">
-      <origin xyz="0 0 0"/>
+   <turtlebot_arm parent="base_arm" color="Gray" gripper_color="Gray" pincher_gripper="true" turtlebot_gripper="false">
+      <origin xyz="0 -0.014 ${AX12_HEIGHT/2 - 0.005}" rpy="0 0 ${M_PI/2}"/>
    </turtlebot_arm>
 </robot>

Commit message: Changed navigation params + arm on top of tb3

File: turtlebot3_description/urdf/turtlebot3_burger.urdf.xacro (robot description, xacro)
@@ -146,5 +146,5 @@
     <parent link="base_link" />
     <child link="base_arm" />
-    <origin xyz="-0.036 0.04 0.2385" rpy="0 0 0"/>
+    <origin xyz="-0.036 0 0.1914" rpy="0 0 0"/>
   </joint>
   <link name="base_arm">
@@ -172,5 +172,5 @@
    <include filename="$(find turtlebot_arm_description)/urdf/$(optenv TURTLEBOT_ARM1 pincher)_arm.urdf.xacro" />
    <turtlebot_arm parent="base_arm" color="Gray" gripper_color="Gray" pincher_gripper="true" turtlebot_gripper="false">
-      <origin xyz="0 -0.014 ${AX12_HEIGHT/2 - 0.005}" rpy="0 0 ${M_PI/2}"/>
+      <origin xyz="0 0.029 0.063" rpy="0 0 ${M_PI/2}"/>
    </turtlebot_arm>
 </robot>
